Commit message: added wheels and joints to the robot - changed the color from blue to black

File: urdf/robot.urdf (robot description, URDF)
Before this commit: robot my_simulation_robot, 2 links, 1 joints
Links:
- added link wheel_left, mass 0.2; collision cylinder length=0.05 radius=0.1; visual cylinder length=0.05 radius=0.1
- added link wheel_right, mass 0.2; collision cylinder length=0.05 radius=0.1; visual cylinder length=0.05 radius=0.1
Joints:
- added joint left_wheel_joint: type continuous, parent base_link, child wheel_left, origin xyz=-0.25 0.3 0 rpy=0 1.5708 0, axis 0 1 0
- added joint right_wheel_joint: type continuous, parent base_link, child wheel_right, origin xyz=-0.25 -0.3 0 rpy=0 1.5708 0, axis 0 1 0

Commit message: wheels were not showing up - fixed errors - robot loads fully in rviz

File: urdf/robot.urdf (robot description, URDF)
Before this commit: robot my_simulation_robot, 4 links, 3 joints
Links:
- removed link wheel_left
- removed link wheel_right
- added link left_wheel, mass 0.2; collision cylinder length=0.05 radius=0.1; visual cylinder length=0.05 radius=0.1
- added link right_wheel, mass 0.2; collision cylinder length=0.05 radius=0.1; visual cylinder length=0.05 radius=0.1
Joints:
- joint left_wheel_joint: child wheel_left -> left_wheel
- joint right_wheel_joint: child wheel_right -> right_wheel

Commit message: fixed robot loading errors - changed base color to lime

File: urdf/robot.urdf (robot description, URDF)
Before this commit: robot simple_robot, 4 links, 3 joints
Links:
- removed link left_wheel
- removed link right_wheel
- added link robot_left_wheel, mass 0.2; collision cylinder length=0.05 radius=0.1; visual cylinder length=0.05 radius=0.1
- added link robot_right_wheel, mass 0.2; collision cylinder length=0.05 radius=0.1; visual cylinder length=0.05 radius=0.1
Joints:
- removed joint left_wheel_joint
- removed joint right_wheel_joint
- added joint robot_left_wheel_joint: type continuous, parent base_link, child robot_left_wheel, origin xyz=-0.25 0.3 0 rpy=0 1.5708 0, axis 0 1 0
- added joint robot_right_wheel_joint: type continuous, parent base_link, child robot_right_wheel, origin xyz=-0.25 -0.3 0 rpy=0 1.5708 0, axis 0 1 0

Commit message: changed the orientation of the base - vertical, to provide more stability - new robot design.

File: urdf/robot.urdf (robot description, URDF)
Before this commit: robot my_simulation_robot, 4 links, 3 joints
Links:
- removed link robot_left_wheel
- removed link robot_right_wheel
- link base_link: geometry collision box size=0.2 0.2 0.5; visual box size=0.2 0.2 0.5
Joints:
- removed joint robot_left_wheel_joint
- removed joint robot_right_wheel_joint

Commit message: added 4 wheels instead of 2 - provides better stability for the robot.

File: urdf/robot.urdf (robot description, URDF)
Before this commit: robot my_simulation_robot, 2 links, 1 joints
Links:
- added link back_left_wheel, mass 0.2; collision cylinder length=0.05 radius=0.05; visual cylinder length=0.05 radius=0.05
- added link back_right_wheel, mass 0.2; collision cylinder length=0.05 radius=0.05; visual cylinder length=0.05 radius=0.05
- added link front_left_wheel, mass 0.2; collision cylinder length=0.05 radius=0.05; visual cylinder length=0.05 radius=0.05
- added link front_right_wheel, mass 0.2; collision cylinder length=0.05 radius=0.05; visual cylinder length=0.05 radius=0.05
Joints:
- added joint back_left_wheel_joint: type continuous, parent base_link, child back_left_wheel, origin xyz=-0.1 0.1 -0.25 rpy=0 1.5708 0, axis 0 1 0
- added joint back_right_wheel_joint: type continuous, parent base_link, child back_right_wheel, origin xyz=-0.1 -0.1 -0.25 rpy=0 1.5708 0, axis 0 1 0
- added joint front_left_wheel_joint: type continuous, parent base_link, child front_left_wheel, origin xyz=0.1 0.1 -0.25 rpy=0 1.5708 0, axis 0 1 0
- added joint front_right_wheel_joint: type continuous, parent base_link, child front_right_wheel, origin xyz=0.1 -0.1 -0.25 rpy=0 1.5708 0, axis 0 1 0

Commit message: added grippers - alignement and asthetic is pending.

File: urdf/robot.urdf (robot description, URDF)
Before this commit: robot my_simulation_robot, 6 links, 5 joints
Links:
- removed link back_left_wheel
- removed link back_right_wheel
- added link gripper, mass 0.05; collision box size=0.1 0.02 0.02; visual box size=0.1 0.02 0.02
- added link gripper_arm, mass 0.1; collision box size=0.3 0.02 0.02; visual box size=0.3 0.02 0.02
- added link rear_left_wheel, mass 0.2; collision cylinder length=0.05 radius=0.05; visual cylinder length=0.05 radius=0.05
- added link rear_right_wheel, mass 0.2; collision cylinder length=0.05 radius=0.05; visual cylinder length=0.05 radius=0.05
Joints:
- removed joint back_left_wheel_joint
- removed joint back_right_wheel_joint
- added joint gripper_arm_joint: type revolute, parent base_link, child gripper_arm, origin xyz=0 0 0.2 rpy=0 0 0, axis 0 1 0, limit lower=-1.5708 upper=1.5708 effort=10 velocity=0.05
- added joint gripper_joint: type prismatic, parent gripper_arm, child gripper, origin xyz=0.3 0 0 rpy=0 0 0, axis 1 0 0, limit lower=0.0 upper=0.1 effort=10 velocity=0.05
- added joint rear_left_wheel_joint: type continuous, parent base_link, child rear_left_wheel, origin xyz=-0.1 0.1 -0.25 rpy=0 1.5708 0, axis 0 1 0
- added joint rear_right_wheel_joint: type continuous, parent base_link, child rear_right_wheel, origin xyz=-0.1 -0.1 -0.25 rpy=0 1.5708 0, axis 0 1 0
